File: pcbs/esp_gamepad/esp_gamepad.kicad_sch (KiCad schematic)
At the start: 55 parts, among them P1 USB_C_Plug_USB2.0, Q1 SI2301DS, SW1 SW_Push, SW10 SW_Push, SW11 SW_Push, SW12 SW_Push, SW13 SW_Push, SW2 SW_Push, SW3 SW_Push, SW4 SW_Push, SW5 SW_Push, SW6 SW_Push, SW7 SW_Push, SW8 SW_Push, SW9 SW_Push, U1 COM-09032, U2 IP5306, U5 LC709203FQH-02TWG, U7 COM-09032

Commit message: gamepad done
Parts:
- removed Q1: SI2301DS, Package_TO_SOT_SMD:TSOT-23, symbol Simulation_SPICE:PMOS
- added C10, C11: 10uF, Capacitor_SMD:C_0805_2012Metric, symbol Device:C
- added J1: 2.54mm, Connector_PinHeader_2.54mm:PinHeader_2x10_P2.54mm_Horizontal, symbol Connector_Generic:Conn_02x10_Counter_Clockwise
- added Q2: SI2300, Package_TO_SOT_SMD:SOT-23_Handsoldering, symbol Simulation_SPICE:NMOS
- added R18, R19: 10K, Resistor_SMD:R_0805_2012Metric, symbol Device:R
- added SW14: DIP, Button_Switch_THT:SW_DIP_SPSTx01_Slide_9.78x4.72mm_W7.62mm_P2.54mm, symbol Switch:SW_SPST
- C5, C6, C7: footprint Capacitor_SMD:C_0805_2012Metric -> Capacitor_Tantalum_SMD:CP_EIA-3528-15_AVX-H_Pad1.50x2.35mm_HandSolder
- L1: footprint (none) -> Inductor_SMD:L_10.4x10.4_H4.8
- P1: footprint (none) -> USB_Type_C:USB_Type_C_6P
- R10: value R -> 2R
- SW1, SW9: footprint (none) -> Button_Switch_THT:SW_PUSH-12mm
- SW10, SW11, SW12, SW13, SW2, SW3, SW4, SW5: footprint (none) -> Keyboard_Switches:SW_MX_LowProfile_Kailh_Choc_V1V2_THT_Hybrid
- SW6, SW8: footprint (none) -> Button_Switch_THT:SW_Tactile_SPST_Angled_PTS645Vx31-2LFS
- SW7: footprint (none) -> Button_Switch_THT:SW_PUSH_6mm
- U2: footprint IP5306_Power_Bank:IP5306_IC -> Package_SO:SOIC-8-1EP_3.9x4.9mm_P1.27mm_EP2.41x3.3mm_ThermalVias
- U3: footprint (none) -> IMU:MPU6050
- U4: footprint (none) -> ESP32_S3_DevkitC1:ESP32_S3_DevkitC1
- U5: footprint Package_DFN_QFN:WDFN-8-1EP_4x3mm_P0.65mm_EP2.4x1.8mm -> Package_DFN_QFN:WDFN-8-1EP_4x3mm_P0.65mm_EP2.4x1.8mm_ThermalVias
- U6: footprint (none) -> LCD_TFT_ST7789:LCD_TFT_1.3_inches_ST7789
Connections:
- net 3V3: now also C10.1, C11.1, J1.1 (Pin_1), J1.20 (Pin_20), R18.2, R19.2
- net CLK: now also J1.14 (Pin_14)
- net GND: now also C10.2, C11.2, J1.10 (Pin_10), J1.19 (Pin_19), J1.2 (Pin_2), Q2.3 (S)
- net IO10: now also J1.15 (Pin_15); no longer R4.1, SW4.1
- net IO11: now also J1.18 (Pin_18); no longer R3.1, SW5.1
- net IO12: now also J1.16 (Pin_16); no longer R1.1, U1.B1A (SEL+)
- net IO13: now also J1.17 (Pin_17); no longer U1.H2 (H)
- net IO14: now also R3.1, SW5.1; no longer U1.V2 (V)
- net IO46: now also R5.1, SW3.1; no longer R6.1, SW2.1
- net IO9: now also R4.1, SW4.1; no longer R5.1, SW3.1
- net MOSI: now also J1.13 (Pin_13)
- net SCL: now also J1.3 (Pin_3), R19.1
- net SDA: now also J1.4 (Pin_4), R18.1
- net VBUS: now also Q2.2 (G)
- net at U4.3 (RST): now also SW14.2 (B)
- net IO37: now reaches U4.34 (IO37)
- net IO37: now also J1.5 (Pin_5)
- net IO4: now reaches U4.4 (IO4)
- net IO4: now also R1.1, U1.B1A (SEL+)
- net IO2: now reaches U4.40 (IO2)
- net IO2: now also J1.6 (Pin_6)
- net IO1: now reaches U4.41 (IO1)
- net IO1: now also J1.7 (Pin_7)
- net RXD: now reaches U4.42 (RXD)
- net RXD: now also J1.8 (Pin_8)
- net TXD: now reaches U4.43 (TXD)
- net TXD: now also J1.9 (Pin_9)
- net IO5: now reaches U4.5 (IO5)
- net IO5: now also U1.H2 (H)
- net IO6: now reaches U4.6 (IO6)
- net IO6: now also U1.V2 (V)
- net IO7: now reaches U4.7 (IO7)
- net IO7: now also R6.1, SW2.1
- net IO15: now reaches U4.8 (IO15)
- net IO15: now also J1.12 (Pin_12)
- net IO16: now reaches U4.9 (IO16)
- net IO16: now also J1.11 (Pin_11)
- new net: Q2.1 (D), SW14.1 (A)
Other:
- note added: "Connector"
- note added: "IMU"
- note removed: "Inertial Measurement Unit"
- moved on the sheet: C8, C9, R1, R13, R14, R15, R16, R17, R3, R4, R5, R6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

Commit message: pcb modification
Parts:
- U1, U7: footprint Joystick:Joystick -> Joystick:PS4_joystick
Connections:
- net GND: now also J1.9 (Pin_9)
- net IO1: now also J1.6 (Pin_6); no longer J1.7 (Pin_7)
- net IO2: now also R11.2, SW8.2; no longer J1.6 (Pin_6)
- net RXD: now also J1.7 (Pin_7); no longer J1.8 (Pin_8)
- net TXD: now also J1.8 (Pin_8); no longer J1.9 (Pin_9)
- net IO39: now reaches R12.2, SW9.2
- net IO39: now also U4.36 (IO39)
Changed lines of the file:
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@@
 	)
 	(junction
+		(at 60.96 187.96)
+		(diameter 0)
+		(color 0 0 0 0)
+	)
+	(junction
 		(at 203.2 139.7)
 		(diameter 0)
@@
 	(wire
 		(pts
+			(xy 60.96 185.42) (xy 60.96 187.96)
+		)
+		(stroke
+			(width 0)
+			(type default)
+		)
+	)
+	(wire
+		(pts
 			(xy 148.59 101.6) (xy 151.13 101.6)
 		)
@@
 	(wire
 		(pts
+			(xy 60.96 187.96) (xy 62.23 187.96)
+		)
+		(stroke
+			(width 0)
+			(type default)
+		)
+	)
+	(wire
+		(pts
 			(xy 162.56 190.5) (xy 160.02 190.5)
 		)
@@
 	(wire
 		(pts
-			(xy 58.42 187.96) (xy 62.23 187.96)
+			(xy 58.42 187.96) (xy 60.96 187.96)
 		)
 		(stroke
@@
 	(wire
 		(pts
+			(xy 62.23 185.42) (xy 60.96 185.42)
+		)
+		(stroke
+			(width 0)
+			(type default)
+		)
+	)
+	(wire
+		(pts
 			(xy 162.56 39.37) (xy 162.56 50.8)
 		)
@@
 	(wire
 		(pts
+			(xy 176.53 116.84) (xy 175.26 116.84)
+		)
+		(stroke
+			(width 0)
+			(type default)
+		)
+	)
+	(wire
+		(pts
 			(xy 54.61 107.95) (xy 43.18 107.95)
 		)
@@
 		)
 	)
-	(label "3V3"
-		(at 162.56 190.5 0)
+	(label "IO39"
+		(at 186.69 78.74 180)
 		(fields_autoplaced yes)
 		(effects
@@
 				(size 1.27 1.27)
 			)
-			(justify left bottom)
+			(justify right bottom)
 		)
 	)
-	(label "IO1"
-		(at 62.23 180.34 180)
+	(label "3V3"
+		(at 162.56 190.5 0)
 		(fields_autoplaced yes)
 		(effects
@@
 				(size 1.27 1.27)
 			)
-			(justify right bottom)
+			(justify left bottom)
 		)
 	)
@@
 		)
 	)
+	(label "RXD"
+		(at 62.23 180.34 180)
+		(fields_autoplaced yes)
+		(effects
+			(font
+				(size 1.27 1.27)
+			)
+			(justify right bottom)
+		)
+	)
 	(label "3V3"
 		(at 252.73 43.18 180)
@@
 		)
 	)
-	(label "IO2"
-		(at 62.23 177.8 180)
-		(fields_autoplaced yes)
-		(effects
-			(font
-				(size 1.27 1.27)
-			)
-			(justify right bottom)
-		)
-	)
 	(label "IO12"
 		(at 149.86 139.7 180)
@@
 		)
 	)
-	(label "RXD"
-		(at 62.23 182.88 180)
-		(fields_autoplaced yes)
-		(effects
-			(font
-				(size 1.27 1.27)
-			)
-			(justify right bottom)
-		)
-	)
 	(label "IO13"
 		(at 149.86 142.24 180)
@@
 		)
 	)
+	(label "TXD"
+		(at 62.23 182.88 180)
+		(fields_autoplaced yes)
+		(effects
+			(font
+				(size 1.27 1.27)
+			)
+			(justify right bottom)
+		)
+	)
 	(label "IO12"
 		(at 74.93 175.26 0)
@@
 		)
 	)
-	(label "TXD"
-		(at 62.23 185.42 180)
-		(fields_autoplaced yes)
-		(effects
-			(font
-				(size 1.27 1.27)
-			)
-			(justify right bottom)
-		)
-	)
 	(label "IO15"
 		(at 74.93 185.42 0)
@@
 		)
 	)
+	(label "IO39"
+		(at 176.53 116.84 0)
+		(fields_autoplaced yes)
+		(effects
+			(font
+				(size 1.27 1.27)
+			)
+			(justify left bottom)
+		)
+	)
 	(label "SCL"
 		(at 199.39 33.02 0)
@@
 		)
 	)
+	(label "IO1"
+		(at 62.23 177.8 180)
+		(fields_autoplaced yes)
+		(effects
+			(font
+				(size 1.27 1.27)
+			)
+			(justify right bottom)
+		)
+	)
 	(label "IO45"
 		(at 176.53 132.08 0)
@@
 		)
 	)
+	(label "IO2"
+		(at 220.98 78.74 180)
+		(fields_autoplaced yes)
+		(effects
+			(font
+				(size 1.27 1.27)
+			)
+			(justify right bottom)
+		)
+	)
 	(label "IO9"
 		(at 106.68 123.19 0)
@@
 			)
 		)
-		(property "Footprint" "Joystick:Joystick"
+		(property "Footprint" "Joystick:PS4_joystick"
 			(at 273.05 125.73 0)
 			(effects
@@
 			)
 		)
-		(property "Footprint" "Joystick:Joystick"
+		(property "Footprint" "Joystick:PS4_joystick"
 			(at 30.48 115.57 0)
 			(effects
