File: pcbs/micromouse/micromouse.kicad_pcb (KiCad board)
At the start: 2 copper layers, 52 parts, among them M1 GA12_N20, M2 GA12_N20, SW1 SW_DPDT_x2, SW2 SW_Push, U2 L7806, U3 AMS1117-5.0

Commit message: 100% done
Parts:
- added C16: 10uF, Capacitor_SMD:C_0805_2012Metric_Pad1.18x1.45mm_HandSolder, B.Cu at (131.3, 134.8)
- added H1: M2, MountingHole:MountingHole_2.2mm_M2, F.Cu at (130.8, 97.5)
- added H2: M2, MountingHole:MountingHole_2.2mm_M2, F.Cu at (130.8, 115.5)
- added H7: M2, MountingHole:MountingHole_2.2mm_M2, F.Cu at (160.4, 97.5)
- added H8: M2, MountingHole:MountingHole_2.2mm_M2, F.Cu at (160.4, 115.5)
- C10, C17, C2, C4, C7, C8, D2, D4, R10, R11, R12, R13, R2, R3, R4, R5, R6, R7, R8, R9, SW2, U1: moved to B.Cu
- M1, M2: footprint N20_DC_Motor:N20_DC_Motor -> XH_2p54:2P_male
- U5, U6, U7, U8, U9: footprint VL53L0X_ToF_Sensor:VL53L0X ToF Sensor -> VL53L0X:VL53L0X_vertical
- moved U7 96.1 mm to (114.3, 57.2), turned to -30 degrees
- moved H4 82.2 mm to (169.0, 78.6)
- moved H6 72.9 mm to (169.0, 134.1)
- moved U4 67.7 mm to (149.5, 93.2)
- moved C12 65.2 mm to (160.8, 73.6)
- moved SW2 62.4 mm to (172.1, 122.4), turned to 90 degrees
- moved C14 62.0 mm to (158.8, 89.4), turned to -90 degrees
- moved U10 60.6 mm to (154.2, 73.7)
- moved M2 58.9 mm to (126.8, 89.3), turned to -90 degrees
- moved U9 58.3 mm to (129.8, 44.5), turned to -60 degrees
- moved SW1 53.7 mm to (132.3, 76.1), turned to -90 degrees
- moved C4 53.3 mm to (165.3, 83.3), turned to 90 degrees
- moved R9 51.8 mm to (167.7, 124.6), turned to 180 degrees
- moved C13 50.8 mm to (143.6, 82.1), turned to -90 degrees
- moved C10 49.4 mm to (163.2, 79.5), turned to -90 degrees
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Connections:
- R10 pad 2: /5V -> /3V3
- U1 pad 12: unconnected-(U1-IO10-Pad12) -> /BAT_ADC
- U1 pad 15: unconnected-(U1-IO13-Pad15) -> /RGB
- U1 pad 3: unconnected-(U1-IO1-Pad3) -> /BUTTON
- U1 pad 4: unconnected-(U1-IO2-Pad4) -> /SCL
- U1 pad 5: unconnected-(U1-IO3-Pad5) -> /SDA
- U1 pad 6: unconnected-(U1-IO4-Pad6) -> /PWM_B
- U1 pad 7: unconnected-(U1-IO5-Pad7) -> /PWM_A
- U4 pad 13: Net-(D4-A) -> Net-(D2-A)
- U4 pad 18: Net-(D4-K) -> Net-(D2-K)
- U4 pad 3: Net-(D2-K) -> Net-(D4-K)
- U4 pad 8: Net-(D2-A) -> Net-(D4-A)
Routing:
- net GND: track 0.00 -> 341.6 mm, vias 0 -> 17
- net /3V3: track 0.00 -> 246.6 mm, vias 0 -> 6
- net /SDA: track 0.00 -> 219.6 mm, vias 0 -> 4
- net /SCL: track 0.00 -> 212.3 mm, vias 0 -> 4
- net /VBAT: track 0.00 -> 115.5 mm, vias 0 -> 1
- net /5V: track 0.00 -> 52.2 mm, vias 0 -> 3
- net /PWM_A: track 0.00 -> 51.7 mm, vias 0 -> 1
- net /6V: track 0.00 -> 43.5 mm, vias 0 -> 2
- net /PWM_B: track 0.00 -> 37.5 mm, vias 0 -> 1
- net Net-(BT1-+): track 0.00 -> 29.2 mm, vias 0 -> 1
- net Net-(D4-A): track 0.00 -> 23.6 mm, vias 0 -> 1
- net /BUTTON: track 0.00 -> 22.1 mm
- net Net-(D4-K): track 0.00 -> 22.0 mm, vias 0 -> 1
- net Net-(D2-A): track 0.00 -> 16.0 mm
- net Net-(D2-K): track 0.00 -> 13.5 mm
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- added copper zone on B.Cu, net GND
- added copper zone on F.Cu, net GND
Other:
- board outline added: 77.4 x 100.8 mm
- board text added: "BATTERY"

Commit message: pcb gerbers done
Parts:
- C12, C13: value 100nF -> 470nF
- C14, C15: value C -> 0.1uF
- C8, C9: value 10uF -> 0.1uF
- moved C15 0.55 mm to (132.8, 89.3)
- moved C6 0.50 mm to (132.8, 85.5)
Routing:
- net /5V: track 52.2 -> 68.8 mm, vias 3 -> 4
- net /VBAT: track 115.5 -> 122.5 mm
- net GND: track 341.6 -> 347.5 mm
